Commit message: urdf updated

File: urdf/my_model.xacro (robot description, xacro)
@@ -1,4 +1,4 @@
 <?xml version="1.0"?>
-<robot name="robot" xmlns:xacro="http://www.ros.org/wiki/xacro">
+<robot xmlns:xacro="http://www.ros.org/wiki/xacro" name="robot">
   <material name="black">
     <color rgba="0.0 0.0 0.0 1.0"/>
@@ -29,11 +29,14 @@
   </gazebo>
   <gazebo reference="link_left_wheel">
-    <material>Gazebo/Green</material>
+    <material>Gazebo/Orange</material>
   </gazebo>
   <gazebo reference="link_right_wheel">
-    <material>Gazebo/Green</material>
+    <material>Gazebo/Orange</material>
   </gazebo>
   <gazebo reference="link_left2_wheel">
-    <material>Gazebo/Green</material>
+    <material>Gazebo/Orange</material>
+  </gazebo>
+  <gazebo reference="camera_link">
+    <material>Gazebo/Blue</material>
   </gazebo>
   <gazebo>
@@ -88,4 +91,76 @@
     </sensor>
   </gazebo>
+   <!--Interial macros-->
+  <xacro:macro name="cylinder_inertia" params="m r h">
+    <inertial>
+      <mass value="${m}"/>
+      <inertia ixx="${m*(3*r*r+h*h)/12}" ixy = "0" ixz = "0" iyy="${m*(3*r*r+h*h)/12}" iyz = "0" izz="${m*r*r/2}"/>
+    </inertial>
+  </xacro:macro>
+  <xacro:macro name="box_inertia" params="m w h d">
+    <inertial>
+      <mass value="${m}"/>
+      <inertia ixx="${m / 12.0 * (d*d + h*h)}" ixy="0.0" ixz="0.0" iyy="${m / 12.0 * (w*w + h*h)}" iyz="0.0" izz="${m / 12.0 * (w*w + d*d)}"/>
+    </inertial>
+  </xacro:macro>
+ <xacro:property name="M_PI" value="3.1415926535897931" />
+  <xacro:macro name="camera_link" params="parent">
+    <link name="camera_link">
+      <collision>
+        <origin xyz="0 0 0.43" rpy="0 0 0" />
+        <geometry>
+          <box size=".1 .1 .1" />
+        </geometry>
+      </collision>
+      <visual>
+        <origin xyz="0 0 0.43" rpy="0 0 0" />
+        <geometry>
+          <box size=".1 .1 .1" />
+        </geometry>
+        <material name="grey">
+            <color rgba="0.2 0.2 0.2 1.0"/>
+        </material>
+      </visual>
+	<xacro:box_inertia m="0.001" w="0.1" h="0.1" d="0.1"/>
+    </link>
+    <joint name="camera_joint" type="fixed">
+        <parent link="${parent}"/>
+        <child link="camera_link"/>
+        <origin rpy="0 0 0" xyz="2.195 0 0.5"/>
+        <axis xyz="1 0 0" />
+    </joint>
+    <gazebo reference="camera_link">
+      <sensor type="camera" name="camera_camera_sensor">
+        <update_rate>30.0</update_rate>
+        <camera>
+          <pose>0.035 0 0.078 0 0 0</pose>
+          <horizontal_fov>${85 * M_PI/180.0}</horizontal_fov>
+          <image>
+            <format>R8G8B8</format>
+            <width>1020</width>
+            <height>1020</height>
+          </image>
+          <clip>
+            <near>0.01</near>
+            <far>100</far>
+          </clip>
+        </camera>
+        <plugin name="camera_camera_controller" filename="libgazebo_ros_camera.so">
+          <alwaysOn>true</alwaysOn>
+          <updateRate>0.0</updateRate>
+          <cameraName>robot_sensor/camera</cameraName>
+          <imageTopicName>image_raw</imageTopicName>
+          <cameraInfoTopicName>camera_info</cameraInfoTopicName>
+          <frameName>camera_link</frameName>
+          <hackBaseline>0.07</hackBaseline>
+          <distortionK1>0.0</distortionK1>
+          <distortionK2>0.0</distortionK2>
+          <distortionK3>0.0</distortionK3>
+          <distortionT1>0.0</distortionT1>
+          <distortionT2>0.0</distortionT2>
+        </plugin>
+      </sensor>
+    </gazebo>
+  </xacro:macro>
 <link name="base_link">
     <inertial>
@@ -108,10 +183,8 @@
     </collision>
   </link>
+  <xacro:camera_link parent="base_link" />
     <link name="link_right_wheel">
-    <inertial>
-      <mass value="2.2"/>
+      <mass value="1"/>
       <origin rpy="0 1.570700 0" xyz="2.195 0 0.27"/>
-    <inertia ixx="0.4" ixy="0.0" ixz="0.0" iyy="0.4" iyz="0.0" izz="0.2"/>
-    </inertial>
     <collision name="link_right_wheel_collision">
 	<geometry>
@@ -124,4 +197,5 @@
 	</geometry>
     </visual>
+    <xacro:cylinder_inertia m="1" r="0.27" h="0.07"/>
   </link>
   <joint name="joint_right_wheel" type="continuous">
@@ -143,9 +217,6 @@
 </transmission>
     <link name="link_left_wheel">
-    <inertial>
-      <mass value="2.2"/>
+      <mass value="1"/>
       <origin rpy="0 1.570700 1.0472" xyz="-1.10000 -1.9 0.27"/>
-      <inertia ixx="0.4" ixy="0.0" ixz="0.0" iyy="0.4" iyz="0.0" izz="0.2"/>
-    </inertial>
     <collision name="link_left_wheel_collision">
 	<geometry>
@@ -158,4 +229,5 @@
 	</geometry>
     </visual>
+    <xacro:cylinder_inertia m="1" r="0.27" h="0.07"/>
   </link>
   <joint name="joint_left_wheel" type="continuous">
@@ -165,10 +237,18 @@
     <axis rpy="0 0 0" xyz="0 0 1"/>
   </joint>
+<!-- Rear wheels transmission -->
+<transmission name="transmission_left_wheel">
+    <type>transmission_interface/SimpleTransmission</type>
+    <joint name="joint_left_wheel">
+        <hardwareInterface>hardware_interface/EffortJointInterface</hardwareInterface>
+    </joint>
+    <actuator name="motor_left_wheel">
+        <hardwareInterface>hardware_interface/EffortJointInterface</hardwareInterface>
+        <mechanicalReduction>1</mechanicalReduction>
+    </actuator>
+</transmission>
     <link name="link_left2_wheel">
-    <inertial>
-      <mass value="2.2"/>
+      <mass value="1"/>
       <origin rpy="0 1.570700 2.0944" xyz="-1.10000 1.9 0.27"/>
-     <inertia ixx="0.4" ixy="0.0" ixz="0.0" iyy="0.4" iyz="0.0" izz="0.2"/>
-    </inertial>
     <collision name="link_left2_wheel_collision">
 	<geometry>
@@ -181,4 +261,5 @@
 	</geometry>
     </visual>
+    <xacro:cylinder_inertia m="1" r="0.27" h="0.07"/>
   </link>
   <joint name="joint_left2_wheel" type="continuous">
@@ -188,3 +269,14 @@
     <axis rpy="0 0 0" xyz="0 0 1"/>
   </joint>
+<!-- Rear wheels transmission -->
+<transmission name="transmission_left2_wheel">
+    <type>transmission_interface/SimpleTransmission</type>
+    <joint name="joint_left2_wheel">
+        <hardwareInterface>hardware_interface/EffortJointInterface</hardwareInterface>
+    </joint>
+    <actuator name="motor_left2_wheel">
+        <hardwareInterface>hardware_interface/EffortJointInterface</hardwareInterface>
+        <mechanicalReduction>1</mechanicalReduction>
+    </actuator>
+</transmission>
 </robot>

Commit message: robot moving is ok--- wheel mass is large --- just camera and sonar added

File: urdf/my_model.xacro (robot description, xacro)
@@ -1,4 +1,27 @@
 <?xml version="1.0"?>
 <robot xmlns:xacro="http://www.ros.org/wiki/xacro" name="robot">
+ <xacro:property name="M_PI" value="3.1415926535897931" />
+ <xacro:property name="rob_scale" value="0.225"/>
+ <xacro:property name="camera_z" value="${rob_scale}"/>
+ <xacro:property name="base_z" value="${rob_scale*0.52}"/>
+<xacro:property name="right_wheel_x" value="${rob_scale*2.195}"/>
+<xacro:property name="right_wheel_y" value="${rob_scale*0}"/>
+<xacro:property name="right_wheel_z" value="${rob_scale*0.27}"/>
+<xacro:property name="right_wheel_length" value="${rob_scale*0.07}"/>
+<xacro:property name="right_wheel_radius" value="${rob_scale*0.27}"/>
+<xacro:property name="right_wheel_mass" value="${rob_scale*100}"/>
+<xacro:property name="left_wheel_x" value="${rob_scale*-1.10000}"/>
+<xacro:property name="left_wheel_y" value="${rob_scale*-1.9}"/>
+<xacro:property name="left_wheel_z" value="${rob_scale*0.27}"/>
+<xacro:property name="left_wheel_length" value="${rob_scale*0.07}"/>
+<xacro:property name="left_wheel_radius" value="${rob_scale*0.27}"/>
+<xacro:property name="left_wheel_mass" value="${rob_scale*100}"/>
+<xacro:property name="left2_wheel_x" value="${rob_scale*-1.10000}"/>
+<xacro:property name="left2_wheel_y" value="${rob_scale*1.9}"/>
+<xacro:property name="left2_wheel_z" value="${rob_scale*0.27}"/>
+<xacro:property name="left2_wheel_length" value="${rob_scale*0.07}"/>
+<xacro:property name="left2_wheel_radius" value="${rob_scale*0.27}"/>
+<xacro:property name="left2_wheel_mass" value="${rob_scale*100}"/>
+<xacro:property name="sensor_size" value="${rob_scale*0.1}"/>
   <material name="black">
     <color rgba="0.0 0.0 0.0 1.0"/>
@@ -39,4 +62,7 @@
   <gazebo reference="camera_link">
     <material>Gazebo/Blue</material>
+  </gazebo>
+    <gazebo reference="sonar_link">
+    <material>Gazebo/Black</material>
   </gazebo>
   <gazebo>
@@ -45,5 +71,5 @@
   </plugin>
 </gazebo>
-  <gazebo>
+<!--   <gazebo>
     <plugin filename="libgazebo_ros_diff_drive.so" name="differential_drive_controller">
       <alwaysOn>true</alwaysOn>
@@ -59,6 +85,6 @@
       <robotBaseFrame>link_chassis</robotBaseFrame>
     </plugin>
-  </gazebo>
-  <gazebo reference="sensor_laser">
+  </gazebo> -->
+<!--   <gazebo reference="sensor_laser">
     <sensor type="ray" name="head_hokuyo_sensor">
       <pose>0 0 0 0 0 0</pose>
@@ -90,5 +116,5 @@
       </plugin>
     </sensor>
-  </gazebo>
+  </gazebo> -->
    <!--Interial macros-->
   <xacro:macro name="cylinder_inertia" params="m r h">
@@ -104,17 +130,15 @@
     </inertial>
   </xacro:macro>
- <xacro:property name="M_PI" value="3.1415926535897931" />
   <xacro:macro name="camera_link" params="parent">
     <link name="camera_link">
+	<origin xyz="${right_wheel_x} ${0} ${camera_z}" rpy="0 0 0" />
       <collision>
-        <origin xyz="0 0 0.43" rpy="0 0 0" />
         <geometry>
-          <box size=".1 .1 .1" />
+          <box size="${sensor_size} ${sensor_size} ${sensor_size}" />
         </geometry>
       </collision>
       <visual>
-        <origin xyz="0 0 0.43" rpy="0 0 0" />
         <geometry>
-          <box size=".1 .1 .1" />
+          <box size="${sensor_size} ${sensor_size} ${sensor_size}" />
         </geometry>
         <material name="grey">
@@ -122,10 +146,10 @@
         </material>
       </visual>
-	<xacro:box_inertia m="0.001" w="0.1" h="0.1" d="0.1"/>
+	<xacro:box_inertia m="0.001" w="${sensor_size}" h="${sensor_size}" d="${sensor_size}"/>
     </link>
     <joint name="camera_joint" type="fixed">
         <parent link="${parent}"/>
         <child link="camera_link"/>
-        <origin rpy="0 0 0" xyz="2.195 0 0.5"/>
+        <origin xyz="${right_wheel_x} ${0} ${camera_z}" rpy="0 0 0" />
         <axis xyz="1 0 0" />
     </joint>
@@ -163,42 +187,121 @@
     </gazebo>
   </xacro:macro>
+  <xacro:macro name="sonar_link" params="parent">
+   <link name="sonar_link">
+        <origin xyz="${left2_wheel_x} ${left2_wheel_y} ${camera_z}" rpy="0 0 ${M_PI/2}" />
+      <collision>
+        <geometry>
+          <box size="${sensor_size} ${sensor_size} ${sensor_size}" />
+        </geometry>
+      </collision>
+      <visual>
+        <geometry>
+          <box size="${sensor_size} ${sensor_size} ${sensor_size}" />
+        </geometry>
+        <material name="grey">
+            <color rgba="0.2 0.2 0.2 1.0"/>
+        </material>
+      </visual>
+	<xacro:box_inertia m="0.001" w="${sensor_size}" h="${sensor_size}" d="${sensor_size}"/>
+  </link>
+     <joint name="sonar_joint" type="fixed">
+        <parent link="${parent}"/>
+        <child link="sonar_link"/>
+        <origin rpy="0 0 ${M_PI/2}" xyz="${left2_wheel_x} ${left2_wheel_y} ${camera_z}"/>
+        <axis xyz="1 0 0" />
+    </joint>
+      <gazebo reference="sonar_link">
+	    <sensor type="ray" name="sonar">
+	  <pose>0.25 0 0 0 0 0</pose>
+	  <update_rate>5</update_rate>
+	  <ray>
+	    <scan>
+	      <horizontal>
+		<samples>5</samples>
+		<resolution>1.0</resolution>
+		<min_angle>-0.25</min_angle>
+		<max_angle>0.25</max_angle>
+	      </horizontal>
+	      <vertical>
+		<samples>5</samples>
+		<resolution>1</resolution>
+		<min_angle>-0.25</min_angle>
+		<max_angle>0.25</max_angle>
+	      </vertical>
+	    </scan>
+	    <range>
+	      <min>0.1</min>
+	      <max>0.5</max>
+	      <resolution>0.01</resolution>
+	    </range>
+	  </ray>
+	  <plugin filename="libgazebo_ros_range.so" name="gazebo_ros_range">
+	    <gaussianNoise>0.005</gaussianNoise>
+	    <alwaysOn>true</alwaysOn>
+	    <updateRate>5</updateRate>
+	    <topicName>sonar</topicName>
+	    <frameName>sonar_link</frameName>
+	    <fov>0.5</fov>
+	    <radiation>ultrasound</radiation>
+	  </plugin>
+	</sensor>
+    </gazebo>
+  </xacro:macro>
 <link name="base_link">
     <inertial>
-      <mass value="20"/>
-      <origin xyz="0 0 0.52" rpy="0 0 3.14"/>
-      <inertia ixx="1.392949" ixy="0" ixz="-0.000108" iyy="1.392846" iyz="-0.000000" izz="-1.000000"/>
+      <mass value="200"/>
+      <origin xyz="0 0 ${base_z}" rpy="0 0 3.14"/>
+      <inertia ixx="0.738" ixy="0" ixz="0" iyy="0.738" iyz="-0.000000" izz="1.304"/>
     </inertial>
 	<visual>
-	<origin xyz="0 0 0.52" rpy="0 0 3.14"/>
-	<geometry>
-        <mesh filename="package://rob_pkg/meshes/two_plate.dae"/>
+	<origin xyz="0 0 ${base_z}" rpy="0 0 3.14"/>
+	<geometry>
+        <mesh filename="package://rob_pkg/meshes/two_plate_s.dae" />
       </geometry>
       <material name="red"/>
     </visual>
     <collision >
-	<origin xyz="0 0 0.52" rpy="0 0 3.14"/>
+	<origin xyz="0 0 ${base_z}" rpy="0 0 3.14"/>
       <geometry>
-        <mesh filename="package://rob_pkg/meshes/two_plate.dae"/>
+        <mesh filename="package://rob_pkg/meshes/two_plate_s.dae"   />
       </geometry>
     </collision>
   </link>
   <xacro:camera_link parent="base_link" />
+  <xacro:sonar_link parent="base_link" />
     <link name="link_right_wheel">
-      <mass value="1"/>
-      <origin rpy="0 1.570700 0" xyz="2.195 0 0.27"/>
+      <mass value="${right_wheel_mass}"/>
+      <origin rpy="0 ${M_PI/2} 0" xyz="${right_wheel_x} ${right_wheel_y} ${right_wheel_z}"/>
     <collision name="link_right_wheel_collision">
 	<geometry>
-	 <cylinder length=".07" radius=".27" />
-	</geometry>
+	 <cylinder length="${right_wheel_length}" radius="${right_wheel_radius}" />
+	</geometry>
+	       <surface>
+                <bounce>
+                    <restitution_coefficient>.2</restitution_coefficient>
+                </bounce>
+                <friction>
+                  <ode>
+                      <mu>1000000</mu>
+                      <mu2>100</mu2>
+                      <fdir1>1 0 0</fdir1>
+                      <slip1> 0</slip1>
+                      <slip2>0</slip2>
+                  </ode>
+                </friction>
+                <contact>
+                  <ode/>
+                </contact>
+            </surface>
     </collision>
     <visual name="link_right_wheel_visual">
 	<geometry>
-	 <cylinder length="0.07" radius="0.27" />
+	 <cylinder length="${right_wheel_length}" radius="${right_wheel_radius}" />
 	</geometry>
     </visual>
-    <xacro:cylinder_inertia m="1" r="0.27" h="0.07"/>
+ <xacro:cylinder_inertia m="${right_wheel_mass}" r="${right_wheel_radius}" h="${right_wheel_length}"/>
   </link>
   <joint name="joint_right_wheel" type="continuous">
-	<origin rpy="0 1.570700 0" xyz="2.195 0 0.27"/>
+	<origin rpy="0 ${M_PI/2} 0" xyz="${right_wheel_x} 0 ${right_wheel_z}"/>
     <child link="link_right_wheel"/>
     <parent link="base_link"/>
@@ -217,20 +320,37 @@
 </transmission>
     <link name="link_left_wheel">
-      <mass value="1"/>
-      <origin rpy="0 1.570700 1.0472" xyz="-1.10000 -1.9 0.27"/>
+      <mass value="${left_wheel_mass}"/>
+      <origin rpy="0 ${M_PI/2} 1.0472" xyz="${left_wheel_x} ${left_wheel_y} ${left_wheel_z}"/>
     <collision name="link_left_wheel_collision">
 	<geometry>
-	 <cylinder length=".07" radius=".27" />
+	 <cylinder length="${left_wheel_length}" radius="${left_wheel_radius}" />
 	</geometry>
     </collision>
     <visual name="link_left_wheel_visual">
 	<geometry>
-	 <cylinder length="0.07" radius="0.27" />
-	</geometry>
+	 <cylinder length="${left_wheel_length}" radius="${left_wheel_radius}" />
+	</geometry>
+	       <surface>
+        <bounce>
+            <restitution_coefficient>.2</restitution_coefficient>
+        </bounce>
+        <friction>
+          <ode>
+              <mu>1000000</mu>
+              <mu2>100</mu2>
+              <fdir1>1 0 0</fdir1>
+              <slip1> 0</slip1>
+              <slip2>0</slip2>
+          </ode>
+        </friction>
+        <contact>
+          <ode/>
+        </contact>
+    </surface>
     </visual>
-    <xacro:cylinder_inertia m="1" r="0.27" h="0.07"/>
+    <xacro:cylinder_inertia m="${right_wheel_mass}" r="${right_wheel_radius}" h="${right_wheel_length}"/>
   </link>
   <joint name="joint_left_wheel" type="continuous">
-  <origin rpy="0 1.570700 1.0472" xyz="-1.10000 -1.9 0.27"/>
+  <origin rpy="0 ${M_PI/2} 1.0472" xyz="${left_wheel_x} ${left_wheel_y} ${left_wheel_z}"/>
     <child link="link_left_wheel"/>
     <parent link="base_link"/>
@@ -249,20 +369,37 @@
 </transmission>
     <link name="link_left2_wheel">
-      <mass value="1"/>
-      <origin rpy="0 1.570700 2.0944" xyz="-1.10000 1.9 0.27"/>
+      <mass value="${left2_wheel_mass}"/>
+      <origin rpy="0 ${M_PI/2} 2.0944" xyz="${left2_wheel_x} ${left2_wheel_y} ${left2_wheel_z}"/>
     <collision name="link_left2_wheel_collision">
 	<geometry>
-	 <cylinder length=".07" radius=".27" />
+	 <cylinder length="${left2_wheel_length}" radius="${left2_wheel_radius}" />
 	</geometry>
     </collision>
     <visual name="link_left2_wheel_visual">
 	<geometry>
-	 <cylinder length="0.07" radius="0.27" />
-	</geometry>
+	 <cylinder length="${left2_wheel_length}" radius="${left2_wheel_radius}" />
+	</geometry>
+	       <surface>
+        <bounce>
+            <restitution_coefficient>.2</restitution_coefficient>
+        </bounce>
+        <friction>
+          <ode>
+              <mu>1000000</mu>
+              <mu2>100</mu2>
+              <fdir1>1 0 0</fdir1>
+              <slip1> 0</slip1>
+              <slip2>0</slip2>
+          </ode>
+        </friction>
+        <contact>
+          <ode/>
+        </contact>
+    </surface>
     </visual>
-    <xacro:cylinder_inertia m="1" r="0.27" h="0.07"/>
+    <xacro:cylinder_inertia m="${right_wheel_mass}" r="${right_wheel_radius}" h="${right_wheel_length}"/>
   </link>
   <joint name="joint_left2_wheel" type="continuous">
-  <origin rpy="0 1.570700 2.0944" xyz="-1.10000 1.9 0.27"/>
+  <origin rpy="0 ${M_PI/2} 2.0944" xyz="${left2_wheel_x} ${left2_wheel_y} ${left2_wheel_z}"/>
     <child link="link_left2_wheel"/>
     <parent link="base_link"/>

Commit message: 1 sonar sensor place fixed

File: urdf/my_model.xacro (robot description, xacro)
@@ -208,5 +208,5 @@
         <parent link="${parent}"/>
         <child link="sonar_link"/>
-        <origin rpy="0 0 ${M_PI/2}" xyz="${left2_wheel_x} ${left2_wheel_y} ${camera_z}"/>
+        <origin rpy="0 0 ${M_PI/2 + M_PI/6}" xyz="${left2_wheel_x} ${left2_wheel_y} ${camera_z}"/>
         <axis xyz="1 0 0" />
     </joint>
@@ -220,17 +220,17 @@
 		<samples>5</samples>
 		<resolution>1.0</resolution>
-		<min_angle>-0.25</min_angle>
-		<max_angle>0.25</max_angle>
+		<min_angle>-0.1</min_angle>
+		<max_angle>0.1</max_angle>
 	      </horizontal>
 	      <vertical>
 		<samples>5</samples>
 		<resolution>1</resolution>
-		<min_angle>-0.25</min_angle>
-		<max_angle>0.25</max_angle>
+		<min_angle>-0.1</min_angle>
+		<max_angle>0.1</max_angle>
 	      </vertical>
 	    </scan>
 	    <range>
-	      <min>0.1</min>
-	      <max>0.5</max>
+	      <min>0.02</min>
+	      <max>1.5</max>
 	      <resolution>0.01</resolution>
 	    </range>

Commit message: three sonar sensors added.

File: urdf/my_model.xacro (robot description, xacro)
@@ -132,5 +132,5 @@
   <xacro:macro name="camera_link" params="parent">
     <link name="camera_link">
-	<origin xyz="${right_wheel_x} ${0} ${camera_z}" rpy="0 0 0" />
+	<origin xyz="${0} ${0} ${camera_z}" rpy="0 0 0" />
       <collision>
         <geometry>
@@ -151,5 +151,5 @@
         <parent link="${parent}"/>
         <child link="camera_link"/>
-        <origin xyz="${right_wheel_x} ${0} ${camera_z}" rpy="0 0 0" />
+        <origin xyz="${0} ${0} ${camera_z}" rpy="0 0 0" />
         <axis xyz="1 0 0" />
     </joint>
@@ -187,7 +187,7 @@
     </gazebo>
   </xacro:macro>
-  <xacro:macro name="sonar_link" params="parent">
-   <link name="sonar_link">
-        <origin xyz="${left2_wheel_x} ${left2_wheel_y} ${camera_z}" rpy="0 0 ${M_PI/2}" />
+  <xacro:macro name="sonar_link_gen" params="parent link_name link_x link_y link_z link_r link_p link_yaw">
+   <link name="${link_name}">
+        <origin xyz="${link_x} ${link_y} ${link_z}" rpy="${link_r} ${link_p} ${link_yaw}" />
       <collision>
         <geometry>
@@ -205,12 +205,12 @@
 	<xacro:box_inertia m="0.001" w="${sensor_size}" h="${sensor_size}" d="${sensor_size}"/>
   </link>
-     <joint name="sonar_joint" type="fixed">
+     <joint name="${link_name}_joint" type="fixed">
         <parent link="${parent}"/>
-        <child link="sonar_link"/>
-        <origin rpy="0 0 ${M_PI/2 + M_PI/6}" xyz="${left2_wheel_x} ${left2_wheel_y} ${camera_z}"/>
+        <child link="${link_name}"/>
+        <origin rpy="${link_r} ${link_p} ${link_yaw}" xyz="${link_x} ${link_y} ${link_z}"/>
         <axis xyz="1 0 0" />
     </joint>
-      <gazebo reference="sonar_link">
-	    <sensor type="ray" name="sonar">
+      <gazebo reference="${link_name}">
+	    <sensor type="ray" name="sonar_${link_name}">
 	  <pose>0.25 0 0 0 0 0</pose>
 	  <update_rate>5</update_rate>
@@ -240,6 +240,6 @@
 	    <alwaysOn>true</alwaysOn>
 	    <updateRate>5</updateRate>
-	    <topicName>sonar</topicName>
-	    <frameName>sonar_link</frameName>
+	    <topicName>sonar_${link_name}</topicName>
+	    <frameName>${link_name}</frameName>
 	    <fov>0.5</fov>
 	    <radiation>ultrasound</radiation>
@@ -269,5 +269,7 @@
   </link>
   <xacro:camera_link parent="base_link" />
-  <xacro:sonar_link parent="base_link" />
+  <xacro:sonar_link_gen parent="base_link" link_name="sonar_link_1" link_x="${left2_wheel_x}" link_y="${left2_wheel_y}" link_z="${camera_z}" link_r="0" link_p="0" link_yaw="${M_PI/2 + M_PI/6}" />
+  <xacro:sonar_link_gen parent="base_link" link_name="sonar_link_2" link_x="${right_wheel_x}" link_y="${right_wheel_y}" link_z="${camera_z}" link_r="0" link_p="0" link_yaw="${0}" />
+  <xacro:sonar_link_gen parent="base_link" link_name="sonar_link_3" link_x="${left_wheel_x}" link_y="${left_wheel_y}" link_z="${camera_z}" link_r="0" link_p="0" link_yaw="${-(M_PI/2 + M_PI/6)}" />
     <link name="link_right_wheel">
       <mass value="${right_wheel_mass}"/>
