Commit message: urdf model friction fixed... simulink obstacle detection added

File: urdf/my_model.xacro (robot description, xacro)
@@ -71,50 +71,28 @@
   </plugin>
 </gazebo>
-<!--   <gazebo>
-    <plugin filename="libgazebo_ros_diff_drive.so" name="differential_drive_controller">
-      <alwaysOn>true</alwaysOn>
-      <updateRate>20</updateRate>
-      <leftJoint>joint_left_wheel</leftJoint>
-      <rightJoint>joint_right_wheel</rightJoint>
-      <wheelSeparation>0.4</wheelSeparation>
-      <wheelDiameter>0.2</wheelDiameter>
-      <torque>0.1</torque>
-      <commandTopic>cmd_vel</commandTopic>
-      <odometryTopic>odom</odometryTopic>
-      <odometryFrame>odom</odometryFrame>
-      <robotBaseFrame>link_chassis</robotBaseFrame>
-    </plugin>
-  </gazebo> -->
-<!--   <gazebo reference="sensor_laser">
-    <sensor type="ray" name="head_hokuyo_sensor">
-      <pose>0 0 0 0 0 0</pose>
-      <visualize>false</visualize>
-      <update_rate>20</update_rate>
-      <ray>
-        <scan>
-          <horizontal>
-            <samples>720</samples>
-            <resolution>1</resolution>
-            <min_angle>-1.570796</min_angle>
-            <max_angle>1.570796</max_angle>
-          </horizontal>
-        </scan>
-        <range>
-          <min>0.10</min>
-          <max>10.0</max>
-          <resolution>0.01</resolution>
-        </range>
-        <noise>
-          <type>gaussian</type>
-          <mean>0.0</mean>
-          <stddev>0.01</stddev>
-        </noise>
-      </ray>
-      <plugin name="gazebo_ros_head_hokuyo_controller" filename="libgazebo_ros_laser.so">
-        <topicName>/m2wr/laser/scan</topicName>
-        <frameName>sensor_laser</frameName>
-      </plugin>
-    </sensor>
-  </gazebo> -->
+     <xacro:macro name="surface_gen" params="main_link_name">
+      <gazebo reference="${main_link_name}">
+      <mu1>500.0</mu1>
+      <mu2>0.0</mu2>
+      <fdir1>1 0 0</fdir1>
+      <maxContacts>1</maxContacts>
+      <minDepth>0.005</minDepth>
+      <gravity>true</gravity>
+     <!--  <surface>
+        <friction>
+          <torsional>
+            <coefficient>10</coefficient>
+            <use_patch_radius>false</use_patch_radius>
+            <surface_radius>0.02175</surface_radius>
+            <patch_radius>0.01</patch_radius>
+          </torsional>
+        </friction>
+        <contact>
+      <poissons_ratio>0.5</poissons_ratio>
+        <elastic_modulus>1e8</elastic_modulus>
+      </contact>
+    </surface> -->
+  </gazebo>
+  </xacro:macro>
    <!--Interial macros-->
   <xacro:macro name="cylinder_inertia" params="m r h">
@@ -250,5 +228,5 @@
 <link name="base_link">
     <inertial>
-      <mass value="200"/>
+      <mass value="10"/>
       <origin xyz="0 0 ${base_z}" rpy="0 0 3.14"/>
       <inertia ixx="0.738" ixy="0" ixz="0" iyy="0.738" iyz="-0.000000" izz="1.304"/>
@@ -279,21 +257,4 @@
 	 <cylinder length="${right_wheel_length}" radius="${right_wheel_radius}" />
 	</geometry>
-	       <surface>
-                <bounce>
-                    <restitution_coefficient>.2</restitution_coefficient>
-                </bounce>
-                <friction>
-                  <ode>
-                      <mu>1000000</mu>
-                      <mu2>100</mu2>
-                      <fdir1>1 0 0</fdir1>
-                      <slip1> 0</slip1>
-                      <slip2>0</slip2>
-                  </ode>
-                </friction>
-                <contact>
-                  <ode/>
-                </contact>
-            </surface>
     </collision>
     <visual name="link_right_wheel_visual">
@@ -304,4 +265,5 @@
  <xacro:cylinder_inertia m="${right_wheel_mass}" r="${right_wheel_radius}" h="${right_wheel_length}"/>
   </link>
+<xacro:surface_gen main_link_name="link_right_wheel"/>
   <joint name="joint_right_wheel" type="continuous">
 	<origin rpy="0 ${M_PI/2} 0" xyz="${right_wheel_x} 0 ${right_wheel_z}"/>
@@ -333,24 +295,8 @@
 	 <cylinder length="${left_wheel_length}" radius="${left_wheel_radius}" />
 	</geometry>
-	       <surface>
-        <bounce>
-            <restitution_coefficient>.2</restitution_coefficient>
-        </bounce>
-        <friction>
-          <ode>
-              <mu>1000000</mu>
-              <mu2>100</mu2>
-              <fdir1>1 0 0</fdir1>
-              <slip1> 0</slip1>
-              <slip2>0</slip2>
-          </ode>
-        </friction>
-        <contact>
-          <ode/>
-        </contact>
-    </surface>
     </visual>
     <xacro:cylinder_inertia m="${right_wheel_mass}" r="${right_wheel_radius}" h="${right_wheel_length}"/>
   </link>
+<xacro:surface_gen main_link_name="link_left_wheel"/>
   <joint name="joint_left_wheel" type="continuous">
   <origin rpy="0 ${M_PI/2} 1.0472" xyz="${left_wheel_x} ${left_wheel_y} ${left_wheel_z}"/>
@@ -382,24 +328,8 @@
 	 <cylinder length="${left2_wheel_length}" radius="${left2_wheel_radius}" />
 	</geometry>
-	       <surface>
-        <bounce>
-            <restitution_coefficient>.2</restitution_coefficient>
-        </bounce>
-        <friction>
-          <ode>
-              <mu>1000000</mu>
-              <mu2>100</mu2>
-              <fdir1>1 0 0</fdir1>
-              <slip1> 0</slip1>
-              <slip2>0</slip2>
-          </ode>
-        </friction>
-        <contact>
-          <ode/>
-        </contact>
-    </surface>
     </visual>
     <xacro:cylinder_inertia m="${right_wheel_mass}" r="${right_wheel_radius}" h="${right_wheel_length}"/>
   </link>
+<xacro:surface_gen main_link_name="link_left2_wheel"/>
   <joint name="joint_left2_wheel" type="continuous">
   <origin rpy="0 ${M_PI/2} 2.0944" xyz="${left2_wheel_x} ${left2_wheel_y} ${left2_wheel_z}"/>

Commit message: model friction fixed

File: urdf/my_model.xacro (robot description, xacro)
@@ -10,5 +10,5 @@
 <xacro:property name="right_wheel_length" value="${rob_scale*0.07}"/>
 <xacro:property name="right_wheel_radius" value="${rob_scale*0.27}"/>
-<xacro:property name="right_wheel_mass" value="${rob_scale*100}"/>
+<xacro:property name="right_wheel_mass" value="${rob_scale*40}"/>
 <xacro:property name="left_wheel_x" value="${rob_scale*-1.10000}"/>
 <xacro:property name="left_wheel_y" value="${rob_scale*-1.9}"/>
@@ -16,5 +16,5 @@
 <xacro:property name="left_wheel_length" value="${rob_scale*0.07}"/>
 <xacro:property name="left_wheel_radius" value="${rob_scale*0.27}"/>
-<xacro:property name="left_wheel_mass" value="${rob_scale*100}"/>
+<xacro:property name="left_wheel_mass" value="${rob_scale*40}"/>
 <xacro:property name="left2_wheel_x" value="${rob_scale*-1.10000}"/>
 <xacro:property name="left2_wheel_y" value="${rob_scale*1.9}"/>
@@ -22,5 +22,5 @@
 <xacro:property name="left2_wheel_length" value="${rob_scale*0.07}"/>
 <xacro:property name="left2_wheel_radius" value="${rob_scale*0.27}"/>
-<xacro:property name="left2_wheel_mass" value="${rob_scale*100}"/>
+<xacro:property name="left2_wheel_mass" value="${rob_scale*40}"/>
 <xacro:property name="sensor_size" value="${rob_scale*0.1}"/>
   <material name="black">
@@ -70,13 +70,36 @@
   <robotNamespace>/robot</robotNamespace>
   </plugin>
+  <plugin name="p3d_base_controller" filename="libgazebo_ros_p3d.so">
+  <alwaysOn>true</alwaysOn>
+  <updateRate>50.0</updateRate>
+  <bodyName>base_link</bodyName>
+  <topicName>odom</topicName>
+  <gaussianNoise>0.01</gaussianNoise>
+  <frameName>world</frameName>
+  <xyzOffsets>0 0 0</xyzOffsets>
+  <rpyOffsets>0 0 0</rpyOffsets>
+</plugin>
 </gazebo>
      <xacro:macro name="surface_gen" params="main_link_name">
       <gazebo reference="${main_link_name}">
-      <mu1>500.0</mu1>
-      <mu2>0.0</mu2>
+      <mu1>5000.0</mu1>
+      <mu2>0</mu2>
       <fdir1>1 0 0</fdir1>
       <maxContacts>1</maxContacts>
       <minDepth>0.005</minDepth>
       <gravity>true</gravity>
+            <surface>
+      <friction>
+      <ode>
+      <slip1>0</slip1>
+      <slip2>0</slip2>
+    </ode>
+              <torsional>
+            <coefficient>1.0</coefficient>
+            <surface_radius>0.5</surface_radius>
+            <use_patch_radius>false</use_patch_radius>
+          </torsional>
+  </friction>
+</surface>
      <!--  <surface>
         <friction>
@@ -226,9 +249,11 @@
     </gazebo>
   </xacro:macro>
+ <link name="dummy">
+   </link>
 <link name="base_link">
     <inertial>
-      <mass value="10"/>
+      <mass value="0.03"/>
       <origin xyz="0 0 ${base_z}" rpy="0 0 3.14"/>
-      <inertia ixx="0.738" ixy="0" ixz="0" iyy="0.738" iyz="-0.000000" izz="1.304"/>
+      <inertia ixx="0.0738" ixy="0" ixz="0" iyy="0.0738" iyz="-0.000000" izz="0.1304"/>
     </inertial>
 	<visual>
@@ -246,4 +271,8 @@
     </collision>
   </link>
+  <joint name="dummy_joint" type="fixed">
+     <parent link="dummy"/>
+     <child link="base_link"/>
+   </joint>
   <xacro:camera_link parent="base_link" />
   <xacro:sonar_link_gen parent="base_link" link_name="sonar_link_1" link_x="${left2_wheel_x}" link_y="${left2_wheel_y}" link_z="${camera_z}" link_r="0" link_p="0" link_yaw="${M_PI/2 + M_PI/6}" />
@@ -285,5 +314,5 @@
     <link name="link_left_wheel">
       <mass value="${left_wheel_mass}"/>
-      <origin rpy="0 ${M_PI/2} 1.0472" xyz="${left_wheel_x} ${left_wheel_y} ${left_wheel_z}"/>
+      <origin rpy="0 ${M_PI/2} ${M_PI/3}" xyz="${left_wheel_x} ${left_wheel_y} ${left_wheel_z}"/>
     <collision name="link_left_wheel_collision">
 	<geometry>
@@ -300,5 +329,5 @@
 <xacro:surface_gen main_link_name="link_left_wheel"/>
   <joint name="joint_left_wheel" type="continuous">
-  <origin rpy="0 ${M_PI/2} 1.0472" xyz="${left_wheel_x} ${left_wheel_y} ${left_wheel_z}"/>
+  <origin rpy="0 ${M_PI/2} ${M_PI/3}" xyz="${left_wheel_x} ${left_wheel_y} ${left_wheel_z}"/>
     <child link="link_left_wheel"/>
     <parent link="base_link"/>
@@ -318,5 +347,5 @@
     <link name="link_left2_wheel">
       <mass value="${left2_wheel_mass}"/>
-      <origin rpy="0 ${M_PI/2} 2.0944" xyz="${left2_wheel_x} ${left2_wheel_y} ${left2_wheel_z}"/>
+      <origin rpy="0 ${M_PI/2} ${M_PI*2/3}" xyz="${left2_wheel_x} ${left2_wheel_y} ${left2_wheel_z}"/>
     <collision name="link_left2_wheel_collision">
 	<geometry>
@@ -333,5 +362,5 @@
 <xacro:surface_gen main_link_name="link_left2_wheel"/>
   <joint name="joint_left2_wheel" type="continuous">
-  <origin rpy="0 ${M_PI/2} 2.0944" xyz="${left2_wheel_x} ${left2_wheel_y} ${left2_wheel_z}"/>
+  <origin rpy="0 ${M_PI/2} ${M_PI*2/3}" xyz="${left2_wheel_x} ${left2_wheel_y} ${left2_wheel_z}"/>
     <child link="link_left2_wheel"/>
     <parent link="base_link"/>

Commit message: sonar sensor place updated... bug2 algorithm updated as well

File: urdf/my_model.xacro (robot description, xacro)
@@ -63,5 +63,11 @@
     <material>Gazebo/Blue</material>
   </gazebo>
-    <gazebo reference="sonar_link">
+    <gazebo reference="sonar_link_1">
+    <material>Gazebo/Black</material>
+  </gazebo>
+    <gazebo reference="sonar_link_2">
+    <material>Gazebo/Black</material>
+  </gazebo>
+    <gazebo reference="sonar_link_3">
     <material>Gazebo/Black</material>
   </gazebo>
@@ -197,13 +203,13 @@
 		<samples>5</samples>
 		<resolution>1.0</resolution>
-		<min_angle>-0.1</min_angle>
-		<max_angle>0.1</max_angle>
+		<min_angle>${-M_PI/12}</min_angle>
+		<max_angle>${+M_PI/12}</max_angle>
 	      </horizontal>
-	      <vertical>
+<!-- 	      <vertical>
 		<samples>5</samples>
 		<resolution>1</resolution>
 		<min_angle>-0.1</min_angle>
 		<max_angle>0.1</max_angle>
-	      </vertical>
+	      </vertical> -->
 	    </scan>
 	    <range>
@@ -252,7 +258,7 @@
    </joint>
   <xacro:camera_link parent="base_link" />
-  <xacro:sonar_link_gen parent="base_link" link_name="sonar_link_1" link_x="${left2_wheel_x}" link_y="${left2_wheel_y}" link_z="${camera_z}" link_r="0" link_p="0" link_yaw="${M_PI/2 + M_PI/6}" />
-  <xacro:sonar_link_gen parent="base_link" link_name="sonar_link_2" link_x="${right_wheel_x}" link_y="${right_wheel_y}" link_z="${camera_z}" link_r="0" link_p="0" link_yaw="${0}" />
-  <xacro:sonar_link_gen parent="base_link" link_name="sonar_link_3" link_x="${left_wheel_x}" link_y="${left_wheel_y}" link_z="${camera_z}" link_r="0" link_p="0" link_yaw="${-(M_PI/2 + M_PI/6)}" />
+  <xacro:sonar_link_gen parent="base_link" link_name="sonar_link_1" link_x="${(left2_wheel_x + left_wheel_x)/1.45}" link_y="${(left2_wheel_y + left_wheel_y)/1.45}" link_z="${right_wheel_z}" link_r="0" link_p="0" link_yaw="${(M_PI)}" />
+  <xacro:sonar_link_gen parent="base_link" link_name="sonar_link_2" link_x="${(right_wheel_x + left_wheel_x)/1.45}" link_y="${(right_wheel_y + left_wheel_y)/1.45}" link_z="${right_wheel_z}" link_r="0" link_p="0" link_yaw="${-(M_PI/3)}" />
+  <xacro:sonar_link_gen parent="base_link" link_name="sonar_link_3" link_x="${(right_wheel_x + left2_wheel_x)/1.45}" link_y="${(right_wheel_y + left2_wheel_y)/1.4}" link_z="${right_wheel_z}" link_r="0" link_p="0" link_yaw="${(M_PI/3)}" />
     <link name="link_right_wheel">
       <mass value="${right_wheel_mass}"/>
